File: GHN626.kicad_sch (KiCad schematic)
At the start: 131 parts, among them SW1 SW_Push_45deg, SW10 SW_Push_45deg, SW11 SW_Push_45deg, SW12 SW_Push_45deg, SW13 SW_Push_45deg, SW14 SW_Push_45deg, SW15 SW_Push_45deg, SW16 SW_Push_45deg, SW17 SW_Push_45deg, SW18 SW_Push_45deg, SW19 SW_Push_45deg, SW2 SW_Push_45deg, SW20 SW_Push_45deg, SW21 SW_Push_45deg, SW22 SW_Push_45deg, SW23 SW_Push_45deg, SW24 SW_Push_45deg, SW25 SW_Push_45deg, SW26 SW_Push_45deg, SW27 SW_Push_45deg, SW28 SW_Push_45deg, SW29 SW_Push_45deg, SW3 SW_Push_45deg, SW30 SW_Push_45deg, SW31 SW_Push_45deg, SW32 SW_Push_45deg, SW33 SW_Push_45deg, SW34 SW_Push_45deg, SW35 SW_Push_45deg, SW36 SW_Push_45deg, SW37 SW_Push_45deg, SW38 SW_Push_45deg, SW39 SW_Push_45deg, SW4 SW_Push_45deg, SW40 SW_Push_45deg, SW41 SW_Push_45deg, SW42 SW_Push_45deg, SW43 SW_Push_45deg, SW44 SW_Push_45deg, SW45 SW_Push_45deg, SW46 SW_Push_45deg, SW47 SW_Push_45deg, SW48 SW_Push_45deg, SW49 SW_Push_45deg, SW5 SW_Push_45deg, SW50 SW_Push_45deg, SW51 SW_Push_45deg, SW52 SW_Push_45deg, SW53 SW_Push_45deg, SW54 SW_Push_45deg, SW55 SW_Push_45deg, SW56 SW_Push_45deg, SW57 SW_Push_45deg, SW58 SW_Push_45deg, SW59 SW_Push_45deg, SW6 SW_Push_45deg, SW60 SW_Push_45deg, SW61 SW_Push_45deg, SW62 SW_Push_45deg, SW7 SW_Push_45deg, SW8 SW_Push_45deg, SW9 SW_Push_45deg, U1 ProMicro

Commit message: base
v1
Parts:
- added BT2: Battery, GHN:custombatteryconnector_small, symbol Device:Battery
Connections:
- net C0: now also U1.12 (B5); no longer U1.24 (B6)
- net C1: now also U1.11 (B4); no longer U1.23 (B2)
- net C10: now also U1.19 (F6); no longer U1.7 (D4)
- net C11: now also U1.20 (F7); no longer U1.8 (C6)
- net C12: now also U1.21 (B1); no longer U1.9 (D7)
- net C2: now also U1.10 (E6); no longer U1.22 (B3)
- net C3: now also U1.9 (D7); no longer U1.21 (B1)
- net C4: now also U1.8 (C6); no longer U1.20 (F7)
- net C5: now also U1.7 (D4); no longer U1.19 (F6)
- net C6: now also U1.6 (D0); no longer U1.18 (F5)
- net C7: now also U1.5 (D1); no longer U1.17 (F4)
- net C8: now also U1.17 (F4); no longer U1.5 (D1)
- net C9: now also U1.18 (F5); no longer U1.6 (D0)
- net GND: now also BT2.2 (-)
- net PSW: now also BT2.1 (+)
- net R2: now also U1.22 (B3); no longer U1.10 (E6)
- net R3: now also U1.23 (B2); no longer U1.11 (B4)
- net R4: now also U1.24 (B6); no longer U1.12 (B5)
Other:
- moved on the sheet: BT1
